File: pcb/pro_micro_hat/pro_micro_hat.sch (KiCad schematic (older format))
At the start: 19 parts, among them U1 ProMicro_2

Commit message: should work
Parts:
- JP1: value Jumper -> D1
- JP10: value Jumper -> F5
- JP11: value Jumper -> F6
- JP12: value Jumper -> F7
- JP13: value Jumper -> B1
- JP14: value Jumper -> B3
- JP15: value Jumper -> B2
- JP16: value Jumper -> B6
- JP2: value Jumper -> D0
- JP3: value Jumper -> D4
- JP4: value Jumper -> D5
- JP5: value Jumper -> D7
- JP6: value Jumper -> E6
- JP7: value Jumper -> B4
- JP8: value Jumper -> B5
- JP9: value Jumper -> F4
- L1, L2: footprint LED_SMD:LED_SK6812_PLCC4_5.0x5.0mm_P3.2mm -> Custom Footies:sk6812_mini_e_reversible
Connections:
- net B1: now also JP13.1
- net F7: now also JP12.1
Changed lines of the file:
@@
 P 5450 1300
 F 0 "JP1" H 5450 1564 50  0000 C CNN
-F 1 "Jumper" H 5450 1473 50  0000 C CNN
+F 1 "D1" H 5450 1473 50  0000 C CNN
 F 2 "Lily58-footprint:Jumper" H 5450 1300 50  0001 C CNN
 F 3 "~" H 5450 1300 50  0001 C CNN
@@
 P 5450 1700
 F 0 "JP2" H 5450 1964 50  0000 C CNN
-F 1 "Jumper" H 5450 1873 50  0000 C CNN
+F 1 "D0" H 5450 1873 50  0000 C CNN
 F 2 "Lily58-footprint:Jumper" H 5450 1700 50  0001 C CNN
 F 3 "~" H 5450 1700 50  0001 C CNN
@@
 P 5450 2050
 F 0 "JP3" H 5450 2314 50  0000 C CNN
-F 1 "Jumper" H 5450 2223 50  0000 C CNN
+F 1 "D4" H 5450 2223 50  0000 C CNN
 F 2 "Lily58-footprint:Jumper" H 5450 2050 50  0001 C CNN
 F 3 "~" H 5450 2050 50  0001 C CNN
@@
 P 5450 2450
 F 0 "JP4" H 5450 2714 50  0000 C CNN
-F 1 "Jumper" H 5450 2623 50  0000 C CNN
+F 1 "D5" H 5450 2623 50  0000 C CNN
 F 2 "Lily58-footprint:Jumper" H 5450 2450 50  0001 C CNN
 F 3 "~" H 5450 2450 50  0001 C CNN
@@
 P 5450 2850
 F 0 "JP5" H 5450 3114 50  0000 C CNN
-F 1 "Jumper" H 5450 3023 50  0000 C CNN
+F 1 "D7" H 5450 3023 50  0000 C CNN
 F 2 "Lily58-footprint:Jumper" H 5450 2850 50  0001 C CNN
 F 3 "~" H 5450 2850 50  0001 C CNN
@@
 P 5450 3200
 F 0 "JP6" H 5450 3464 50  0000 C CNN
-F 1 "Jumper" H 5450 3373 50  0000 C CNN
+F 1 "E6" H 5450 3373 50  0000 C CNN
 F 2 "Lily58-footprint:Jumper" H 5450 3200 50  0001 C CNN
 F 3 "~" H 5450 3200 50  0001 C CNN
@@
 P 5450 3550
 F 0 "JP7" H 5450 3814 50  0000 C CNN
-F 1 "Jumper" H 5450 3723 50  0000 C CNN
+F 1 "B4" H 5450 3723 50  0000 C CNN
 F 2 "Lily58-footprint:Jumper" H 5450 3550 50  0001 C CNN
 F 3 "~" H 5450 3550 50  0001 C CNN
@@
 P 5450 3950
 F 0 "JP8" H 5450 4214 50  0000 C CNN
-F 1 "Jumper" H 5450 4123 50  0000 C CNN
+F 1 "B5" H 5450 4123 50  0000 C CNN
 F 2 "Lily58-footprint:Jumper" H 5450 3950 50  0001 C CNN
 F 3 "~" H 5450 3950 50  0001 C CNN
@@
 P 7250 1300
 F 0 "JP9" H 7250 1564 50  0000 C CNN
-F 1 "Jumper" H 7250 1473 50  0000 C CNN
+F 1 "F4" H 7250 1473 50  0000 C CNN
 F 2 "Lily58-footprint:Jumper" H 7250 1300 50  0001 C CNN
 F 3 "~" H 7250 1300 50  0001 C CNN
@@
 P 7250 1700
 F 0 "JP10" H 7250 1964 50  0000 C CNN
-F 1 "Jumper" H 7250 1873 50  0000 C CNN
+F 1 "F5" H 7250 1873 50  0000 C CNN
 F 2 "Lily58-footprint:Jumper" H 7250 1700 50  0001 C CNN
 F 3 "~" H 7250 1700 50  0001 C CNN
@@
 P 7250 2050
 F 0 "JP11" H 7250 2314 50  0000 C CNN
-F 1 "Jumper" H 7250 2223 50  0000 C CNN
+F 1 "F6" H 7250 2223 50  0000 C CNN
 F 2 "Lily58-footprint:Jumper" H 7250 2050 50  0001 C CNN
 F 3 "~" H 7250 2050 50  0001 C CNN
@@
 P 7250 2450
 F 0 "JP12" H 7250 2714 50  0000 C CNN
-F 1 "Jumper" H 7250 2623 50  0000 C CNN
+F 1 "F7" H 7250 2623 50  0000 C CNN
 F 2 "Lily58-footprint:Jumper" H 7250 2450 50  0001 C CNN
 F 3 "~" H 7250 2450 50  0001 C CNN
@@
 P 7250 2850
 F 0 "JP13" H 7250 3114 50  0000 C CNN
-F 1 "Jumper" H 7250 3023 50  0000 C CNN
+F 1 "B1" H 7250 3023 50  0000 C CNN
 F 2 "Lily58-footprint:Jumper" H 7250 2850 50  0001 C CNN
 F 3 "~" H 7250 2850 50  0001 C CNN
@@
 P 7250 3200
 F 0 "JP14" H 7250 3464 50  0000 C CNN
-F 1 "Jumper" H 7250 3373 50  0000 C CNN
+F 1 "B3" H 7250 3373 50  0000 C CNN
 F 2 "Lily58-footprint:Jumper" H 7250 3200 50  0001 C CNN
 F 3 "~" H 7250 3200 50  0001 C CNN
@@
 P 7250 3550
 F 0 "JP15" H 7250 3814 50  0000 C CNN
-F 1 "Jumper" H 7250 3723 50  0000 C CNN
+F 1 "B2" H 7250 3723 50  0000 C CNN
 F 2 "Lily58-footprint:Jumper" H 7250 3550 50  0001 C CNN
 F 3 "~" H 7250 3550 50  0001 C CNN
@@
 P 7250 3950
 F 0 "JP16" H 7250 4214 50  0000 C CNN
-F 1 "Jumper" H 7250 4123 50  0000 C CNN
+F 1 "B6" H 7250 4123 50  0000 C CNN
 F 2 "Lily58-footprint:Jumper" H 7250 3950 50  0001 C CNN
 F 3 "~" H 7250 3950 50  0001 C CNN
@@
 F 0 "L1" H 6200 5262 51  0000 C CNN
 F 1 "SK6812MINI" H 6200 5197 16  0000 C CNN
-F 2 "LED_SMD:LED_SK6812_PLCC4_5.0x5.0mm_P3.2mm" H 6200 5000 60  0001 C CNN
+F 2 "Custom Footies:sk6812_mini_e_reversible" H 6200 5000 60  0001 C CNN
 F 3 "" H 6200 5000 60  0001 C CNN
 	1    6200 5000
@@
 F 0 "L2" H 6200 5762 51  0000 C CNN
 F 1 "SK6812MINI" H 6200 5697 16  0000 C CNN
-F 2 "LED_SMD:LED_SK6812_PLCC4_5.0x5.0mm_P3.2mm" H 6200 5500 60  0001 C CNN
+F 2 "Custom Footies:sk6812_mini_e_reversible" H 6200 5500 60  0001 C CNN
 F 3 "" H 6200 5500 60  0001 C CNN
 	1    6200 5500
@@
 Text GLabel 6950 2050 0    50   Input ~ 0
 F6
-Text GLabel 6950 2400 0    50   Input ~ 0
+Text GLabel 6950 2450 0    50   Input ~ 0
 F7
-Text GLabel 6950 2800 0    50   Input ~ 0
+Text GLabel 6950 2850 0    50   Input ~ 0
 B1
 Text GLabel 6950 3200 0    50   Input ~ 0
